Commit message: Child link sepcyfies origin

File: model/leg.urdf.xacro (robot description, xacro)
@@ -64,5 +64,5 @@
         <xacro:if value="${not (parent_name == 'base_link')}">
           <parent link="${leg_prefix}_${parent['name']}"/>
-          <origin xyz="${parent['joint']['origin'][0]}"
+          <origin xyz="${child['joint']['origin'][0]}"
                   rpy="0 0 0"/>
         </xacro:if>

Commit message: one more save

File: model/leg.urdf.xacro (robot description, xacro)
@@ -6,9 +6,9 @@
     <xacro:property name="robot_props" value="${load_yaml(yaml_file)}" />
     <!-- CONDITIONAL BLOCKS -->
-    <xacro:if value="${reflect}"> <xacro:property name="reflect_multiplier" value="-1" /> </xacro:if>
-    <xacro:if value="${not reflect}"> <xacro:property name="reflect_multiplier" value="1" />   </xacro:if>
-    <xacro:if value="${leg_pos=='rear'}"> <xacro:property name="leg_pos_val" value="${-robot_props['body']['link']['length']/2}" /> </xacro:if>
+    <xacro:if value="${reflect}"> <xacro:property name="reflect_multiplier" value="1" /> </xacro:if>
+    <xacro:if value="${not reflect}"> <xacro:property name="reflect_multiplier" value="-1" />   </xacro:if>
+    <xacro:if value="${leg_pos=='rear'}"> <xacro:property name="leg_pos_val" value="${-robot_props['body']['length']/2}" /> </xacro:if>
     <xacro:if value="${leg_pos=='central'}"> <xacro:property name="leg_pos_val" value="0" /> </xacro:if>
-    <xacro:if value="${leg_pos=='front'}"> <xacro:property name="leg_pos_val" value="${robot_props['body']['link']['length']/2}" /> </xacro:if>
+    <xacro:if value="${leg_pos=='front'}"> <xacro:property name="leg_pos_val" value="${robot_props['body']['length']/2}" /> </xacro:if>
     <!-- LEG LINK -->
     <xacro:macro name="leg_link" params="props">
@@ -16,31 +16,9 @@
         <visual>
           <geometry>
-            <xacro:property name="mesh_file" value="${props['link']['mesh_file']}" />
-            <xacro:if value="${mesh_file == 'None'}">
-              <cylinder length="${props['link']['length']}"
-                        radius="${props['link']['radius']}" />
-            </xacro:if>
-            <xacro:if value="${mesh_file != 'None'}">
-              <mesh filename="${mesh_file}" scale="1 1 1" />
-            </xacro:if>
-            <!-- <material name="${props['link']['material']}"/> -->
+            <cylinder length="${props['link']['length']}"
+                      radius="${props['link']['radius']}" />
           </geometry>
-          <xacro:property name="props_name" value="${props['name']}" />
-          <xacro:if value="${props_name == 'coxa'}">
-            <origin rpy="${props['link']['rpy'][0]}
-                         ${props['link']['rpy'][1]}
-                         ${props['link']['rpy'][2]}"
-                    xyz="${props['link']['origin'][0]}
-                         ${props['link']['origin'][1]*reflect_multiplier}
-                         ${props['link']['origin'][2]}"/>
-          </xacro:if>
-          <xacro:if value="${props_name != 'coxa'}">
-            <origin xyz="${props['link']['origin'][0]}
-                         ${props['link']['origin'][1]}
-                         ${props['link']['origin'][2]}"
-                    rpy="${props['link']['rpy'][0]}
-                         ${props['link']['rpy'][1]}
-                         ${props['link']['rpy'][2]}"/>
-          </xacro:if>
+          <origin xyz="0 0 -${props['link']['length']/2}"
+                  rpy="0 0 ${pi/2}" />
         </visual>
         <collision>
@@ -52,11 +30,11 @@
         </collision>
         <inertial>
-          <mass value="${props['inertial']['mass']}" />
-          <inertia ixx="${props['inertial']['inertia']['ixx']}"
-                   ixy="${props['inertial']['inertia']['ixy']}"
-                   ixz="${props['inertial']['inertia']['ixz']}"
-                   iyy="${props['inertial']['inertia']['iyy']}"
-                   iyz="${props['inertial']['inertia']['iyz']}"
-                   izz="${props['inertial']['inertia']['izz']}" />
+          <mass value="${props['link']['mass']}" />
+          <inertia ixx="${props['link']['inertia']['ixx']}"
+                   ixy="${props['link']['inertia']['ixy']}"
+                   ixz="${props['link']['inertia']['ixz']}"
+                   iyy="${props['link']['inertia']['iyy']}"
+                   iyz="${props['link']['inertia']['iyz']}"
+                   izz="${props['link']['inertia']['izz']}" />
         </inertial>
       </link>
@@ -70,5 +48,5 @@
           <parent link="base_link" />
           <origin xyz="${leg_pos_val}
-                       ${reflect_multiplier*robot_props['body']['link']['width']/2}
+                       ${reflect_multiplier*robot_props['body']['width']/2}
                        0"
                   rpy="${reflect_multiplier*pi/2} 0 0" />
@@ -76,7 +54,5 @@
         <xacro:if value="${not (parent_name == 'base_link')}">
           <parent link="${leg_prefix}_${parent['name']}" />
-          <origin xyz="${child['joint']['origin'][0]}
-                       ${child['joint']['origin'][1]}
-                       ${child['joint']['origin'][2]}"
+          <origin xyz="${child['joint']['origin'][0]}"
                   rpy="0 0 0" />
         </xacro:if>
