Commit message: Leg transmition

File: model/body.urdf.xacro (robot description, xacro)
@@ -8,5 +8,7 @@
       <visual>
         <geometry>
-          <box size="${props['body']['length']} ${props['body']['width']} ${props['body']['thickness']}" />
+          <box size="${props['body']['length']}
+                     ${props['body']['width']}
+                     ${props['body']['thickness']}" />
         </geometry>
         <origin xyz="0 0 0" />
@@ -14,5 +16,7 @@
       <collision>
         <geometry>
-          <box size="${props['body']['length']} ${props['body']['width']} ${props['body']['thickness']}" />
+          <box size="${props['body']['length']}
+                     ${props['body']['width']}
+                     ${props['body']['thickness']}" />
         </geometry>
       </collision>

File: model/leg.urdf.xacro (robot description, xacro)
@@ -5,20 +5,10 @@
     <xacro:property name="yaml_file" value="${props_path}" />
     <xacro:property name="robot_props" value="${load_yaml(yaml_file)}" />
-    <!-- coditional blocks -->
-    <xacro:if value="${reflect}">
-      <xacro:property name="reflect_multiplier" value="1" scope="parent" />
-    </xacro:if>
-    <xacro:if value="${not reflect}">
-      <xacro:property name="reflect_multiplier" value="-1" scope="parent" />
-    </xacro:if>
-    <xacro:if value="${leg_pos == 'rear'}">
-      <xacro:property name="leg_pos" value="${-robot_props['body']['length']/2}" scope="parent" />
-    </xacro:if>
-    <xacro:if value="${leg_pos == 'central'}">
-      <xacro:property name="leg_pos" value="0" scope="parent" />
-    </xacro:if>
-    <xacro:if value="${leg_pos == 'front'}">
-      <xacro:property name="leg_pos" value="${robot_props['body']['length']/2}" scope="parent" />
-    </xacro:if>
+    <!-- CONDITIONAL BLOCKS -->
+    <xacro:if value="${reflect}"> <xacro:property name="reflect_multiplier" value="1" /> </xacro:if>
+    <xacro:if value="${not reflect}"> <xacro:property name="reflect_multiplier" value="-1" />   </xacro:if>
+    <xacro:if value="${leg_pos=='rear'}"> <xacro:property name="leg_pos_val" value="${-robot_props['body']['length']/2}" /> </xacro:if>
+    <xacro:if value="${leg_pos=='central'}"> <xacro:property name="leg_pos_val" value="0" /> </xacro:if>
+    <xacro:if value="${leg_pos=='front'}"> <xacro:property name="leg_pos_val" value="${robot_props['body']['length']/2}" /> </xacro:if>
     <!-- LEG LINK -->
     <xacro:macro name="leg_link" params="props">
@@ -57,5 +47,5 @@
         <xacro:if value="${parent_name == 'base_link'}">
           <parent link="base_link" />
-          <origin xyz="${leg_pos}
+          <origin xyz="${leg_pos_val}
                        ${reflect_multiplier*robot_props['body']['width']/2}
                        0"
@@ -76,4 +66,16 @@
                velocity="${robot_props['servo']['velocity']}" />
       </joint>
+      <!-- TRANSMITION DEFINITION -->
+      <transmission name="${leg_prefix}_${parent['name']}_to_${child['name']}_transmition"
+                    type="SimpleTransmission">
+        <type>transmission_interface/SimpleTransmission</type>
+        <joint name="${leg_prefix}_${parent['name']}_to_${child['name']}_joint">
+          <hardwareInterface>EffortJointInterface</hardwareInterface>
+        </joint>
+        <actuator name="${leg_prefix}_${parent['name']}_to_${child['name']}_actuator">
+          <hardwareInterface>EffortJointInterface</hardwareInterface>
+          <mechanicalReduction>1</mechanicalReduction>
+        </actuator>
+      </transmission>
     </xacro:macro>
     <!-- DEFINE LINKS -->

Commit message: OBJ, robot phisical properties

File: model/body.urdf.xacro (robot description, xacro)
@@ -8,25 +8,34 @@
       <visual>
         <geometry>
-          <box size="${props['body']['length']}
-                     ${props['body']['width']}
-                     ${props['body']['thickness']}" />
+          <xacro:property name="mesh_file" value="${props['body']['link']['mesh_file']}" />
+          <xacro:if value="${mesh_file == 'None'}">
+            <box size="${props['body']['link']['length']}
+                       ${props['body']['link']['width']}
+                       ${props['body']['link']['thickness']}" />
+          </xacro:if>
+          <xacro:if value="${mesh_file != 'None'}">
+            <mesh filename="${mesh_file}" />
+          </xacro:if>
         </geometry>
-        <origin xyz="0 0 0" />
+        <origin xyz="0 0 0"
+                rpy="${props['body']['link']['rpy'][0]}"/>
       </visual>
       <collision>
         <geometry>
-          <box size="${props['body']['length']}
-                     ${props['body']['width']}
-                     ${props['body']['thickness']}" />
+          <box size="${props['body']['link']['length']}
+                     ${props['body']['link']['width']}
+                     ${props['body']['link']['thickness']}" />
         </geometry>
       </collision>
       <inertial>
-        <mass value="${props['body']['mass']}" />
-        <inertia ixx="${props['body']['inertia']['ixx']}"
-                 ixy="${props['body']['inertia']['ixy']}"
-                 ixz="${props['body']['inertia']['ixz']}"
-                 iyy="${props['body']['inertia']['iyy']}"
-                 iyz="${props['body']['inertia']['iyz']}"
-                 izz="${props['body']['inertia']['izz']}" />
+        <mass value="${props['body']['inertial']['mass']}" />
+        <inertia ixx="${props['body']['inertial']['inertia']['ixx']}"
+                 ixy="${props['body']['inertial']['inertia']['ixy']}"
+                 ixz="${props['body']['inertial']['inertia']['ixz']}"
+                 iyy="${props['body']['inertial']['inertia']['iyy']}"
+                 iyz="${props['body']['inertial']['inertia']['iyz']}"
+                 izz="${props['body']['inertial']['inertia']['izz']}" />
+         <origin xyz="${props['body']['inertial']['origin'][0]}"
+                 rpy="0 0 0" />
       </inertial>
     </link>

File: model/leg.urdf.xacro (robot description, xacro)
@@ -8,7 +8,7 @@
     <xacro:if value="${reflect}"> <xacro:property name="reflect_multiplier" value="1" /> </xacro:if>
     <xacro:if value="${not reflect}"> <xacro:property name="reflect_multiplier" value="-1" />   </xacro:if>
-    <xacro:if value="${leg_pos=='rear'}"> <xacro:property name="leg_pos_val" value="${-robot_props['body']['length']/2}" /> </xacro:if>
+    <xacro:if value="${leg_pos=='rear'}"> <xacro:property name="leg_pos_val" value="${-robot_props['body']['link']['length']/2}" /> </xacro:if>
     <xacro:if value="${leg_pos=='central'}"> <xacro:property name="leg_pos_val" value="0" /> </xacro:if>
-    <xacro:if value="${leg_pos=='front'}"> <xacro:property name="leg_pos_val" value="${robot_props['body']['length']/2}" /> </xacro:if>
+    <xacro:if value="${leg_pos=='front'}"> <xacro:property name="leg_pos_val" value="${robot_props['body']['link']['length']/2}" /> </xacro:if>
     <!-- LEG LINK -->
     <xacro:macro name="leg_link" params="props">
@@ -30,11 +30,11 @@
         </collision>
         <inertial>
-          <mass value="${props['link']['mass']}" />
-          <inertia ixx="${props['link']['inertia']['ixx']}"
-                   ixy="${props['link']['inertia']['ixy']}"
-                   ixz="${props['link']['inertia']['ixz']}"
-                   iyy="${props['link']['inertia']['iyy']}"
-                   iyz="${props['link']['inertia']['iyz']}"
-                   izz="${props['link']['inertia']['izz']}" />
+          <mass value="${props['inertial']['mass']}" />
+          <inertia ixx="${props['inertial']['inertia']['ixx']}"
+                   ixy="${props['inertial']['inertia']['ixy']}"
+                   ixz="${props['inertial']['inertia']['ixz']}"
+                   iyy="${props['inertial']['inertia']['iyy']}"
+                   iyz="${props['inertial']['inertia']['iyz']}"
+                   izz="${props['inertial']['inertia']['izz']}" />
         </inertial>
       </link>
@@ -48,5 +48,5 @@
           <parent link="base_link" />
           <origin xyz="${leg_pos_val}
-                       ${reflect_multiplier*robot_props['body']['width']/2}
+                       ${reflect_multiplier*robot_props['body']['link']['width']/2}
                        0"
                   rpy="${reflect_multiplier*pi/2} 0 0" />

File: robot.urdf (robot description, URDF)
Before this commit: robot hexapod, 19 links, 18 joints
Links:
- link base_link: mass 10 -> 0.12138; geometry collision box size=0.3618 0.136 0.052; visual box size=0.3618 0.136 0.052
- link left_central_coxa: mass 0.2 -> 0.12138; geometry collision sphere radius=0.016; visual cylinder length=0.036 radius=0.016
- link left_central_femur: mass 0.2 -> 0.02696; geometry collision sphere radius=0.02; visual cylinder length=0.055 radius=0.02
- link left_central_tibia: mass 0.2 -> 0.08473; geometry collision sphere radius=0.13; visual cylinder length=0.1633 radius=0.13
- link left_front_coxa: mass 0.2 -> 0.12138; geometry collision sphere radius=0.016; visual cylinder length=0.036 radius=0.016
- link left_front_femur: mass 0.2 -> 0.02696; geometry collision sphere radius=0.02; visual cylinder length=0.055 radius=0.02
- link left_front_tibia: mass 0.2 -> 0.08473; geometry collision sphere radius=0.13; visual cylinder length=0.1633 radius=0.13
- link left_rear_coxa: mass 0.2 -> 0.12138; geometry collision sphere radius=0.016; visual cylinder length=0.036 radius=0.016
- link left_rear_femur: mass 0.2 -> 0.02696; geometry collision sphere radius=0.02; visual cylinder length=0.055 radius=0.02
- link left_rear_tibia: mass 0.2 -> 0.08473; geometry collision sphere radius=0.13; visual cylinder length=0.1633 radius=0.13
- link right_central_coxa: mass 0.2 -> 0.12138; geometry collision sphere radius=0.016; visual cylinder length=0.036 radius=0.016
- link right_central_femur: mass 0.2 -> 0.02696; geometry collision sphere radius=0.02; visual cylinder length=0.055 radius=0.02
- link right_central_tibia: mass 0.2 -> 0.08473; geometry collision sphere radius=0.13; visual cylinder length=0.1633 radius=0.13
- link right_front_coxa: mass 0.2 -> 0.12138; geometry collision sphere radius=0.016; visual cylinder length=0.036 radius=0.016
- link right_front_femur: mass 0.2 -> 0.02696; geometry collision sphere radius=0.02; visual cylinder length=0.055 radius=0.02
- link right_front_tibia: mass 0.2 -> 0.08473; geometry collision sphere radius=0.13; visual cylinder length=0.1633 radius=0.13
- link right_rear_coxa: mass 0.2 -> 0.12138; geometry collision sphere radius=0.016; visual cylinder length=0.036 radius=0.016
- link right_rear_femur: mass 0.2 -> 0.02696; geometry collision sphere radius=0.02; visual cylinder length=0.055 radius=0.02
- link right_rear_tibia: mass 0.2 -> 0.08473; geometry collision sphere radius=0.13; visual cylinder length=0.1633 radius=0.13
Joints:
- joint left_central_base_link_to_coxa_joint: origin xyz=0                        0.075                        0 rpy=1.57079632679 0 0 -> xyz=0                        0.068                        0 rpy=1.57079632679 0 0
- joint left_front_base_link_to_coxa_joint: origin xyz=0.15                        0.075                        0 rpy=1.57079632679 0 0 -> xyz=0.1809                        0.068                        0 rpy=1.57079632679 0 0
- joint left_rear_base_link_to_coxa_joint: origin xyz=-0.15                        0.075                        0 rpy=1.57079632679 0 0 -> xyz=-0.1809                        0.068                        0 rpy=1.57079632679 0 0
- joint right_central_base_link_to_coxa_joint: origin xyz=0                        -0.075                        0 rpy=-1.57079632679 0 0 -> xyz=0                        -0.068                        0 rpy=-1.57079632679 0 0
- joint right_front_base_link_to_coxa_joint: origin xyz=0.15                        -0.075                        0 rpy=-1.57079632679 0 0 -> xyz=0.1809                        -0.068                        0 rpy=-1.57079632679 0 0
- joint right_rear_base_link_to_coxa_joint: origin xyz=-0.15                        -0.075                        0 rpy=-1.57079632679 0 0 -> xyz=-0.1809                        -0.068                        0 rpy=-1.57079632679 0 0

Commit message: reversing old stuff

File: model/body.urdf.xacro (robot description, xacro)
@@ -15,9 +15,14 @@
           </xacro:if>
           <xacro:if value="${mesh_file != 'None'}">
-            <mesh filename="${mesh_file}" />
+            <mesh filename="${mesh_file}" scale="1 1 1" />
           </xacro:if>
+          <!-- <material name="${props['body']['link']['material']}"/> -->
         </geometry>
-        <origin xyz="0 0 0"
-                rpy="${props['body']['link']['rpy'][0]}"/>
+        <origin xyz="${props['body']['link']['origin'][0]}
+                     ${props['body']['link']['origin'][1]}
+                     ${props['body']['link']['origin'][2]}"
+                rpy="${props['body']['link']['rpy'][0]}
+                     ${props['body']['link']['rpy'][1]}
+                     ${props['body']['link']['rpy'][2]}"/>
       </visual>
       <collision>
@@ -36,5 +41,7 @@
                  iyz="${props['body']['inertial']['inertia']['iyz']}"
                  izz="${props['body']['inertial']['inertia']['izz']}" />
-         <origin xyz="${props['body']['inertial']['origin'][0]}"
+         <origin xyz="${props['body']['inertial']['origin'][0]}
+                      ${props['body']['inertial']['origin'][1]}
+                      ${props['body']['inertial']['origin'][2]}"
                  rpy="0 0 0" />
       </inertial>

File: model/leg.urdf.xacro (robot description, xacro)
@@ -6,6 +6,6 @@
     <xacro:property name="robot_props" value="${load_yaml(yaml_file)}" />
     <!-- CONDITIONAL BLOCKS -->
-    <xacro:if value="${reflect}"> <xacro:property name="reflect_multiplier" value="1" /> </xacro:if>
-    <xacro:if value="${not reflect}"> <xacro:property name="reflect_multiplier" value="-1" />   </xacro:if>
+    <xacro:if value="${reflect}"> <xacro:property name="reflect_multiplier" value="-1" /> </xacro:if>
+    <xacro:if value="${not reflect}"> <xacro:property name="reflect_multiplier" value="1" />   </xacro:if>
     <xacro:if value="${leg_pos=='rear'}"> <xacro:property name="leg_pos_val" value="${-robot_props['body']['link']['length']/2}" /> </xacro:if>
     <xacro:if value="${leg_pos=='central'}"> <xacro:property name="leg_pos_val" value="0" /> </xacro:if>
@@ -16,9 +16,31 @@
         <visual>
           <geometry>
-            <cylinder length="${props['link']['length']}"
-                      radius="${props['link']['radius']}" />
+            <xacro:property name="mesh_file" value="${props['link']['mesh_file']}" />
+            <xacro:if value="${mesh_file == 'None'}">
+              <cylinder length="${props['link']['length']}"
+                        radius="${props['link']['radius']}" />
+            </xacro:if>
+            <xacro:if value="${mesh_file != 'None'}">
+              <mesh filename="${mesh_file}" scale="1 1 1" />
+            </xacro:if>
+            <!-- <material name="${props['link']['material']}"/> -->
           </geometry>
-          <origin xyz="0 0 -${props['link']['length']/2}"
-                  rpy="0 0 ${pi/2}" />
+          <xacro:property name="props_name" value="${props['name']}" />
+          <xacro:if value="${props_name == 'coxa'}">
+            <origin rpy="${props['link']['rpy'][0]}
+                         ${props['link']['rpy'][1]}
+                         ${props['link']['rpy'][2]}"
+                    xyz="${props['link']['origin'][0]}
+                         ${props['link']['origin'][1]*reflect_multiplier}
+                         ${props['link']['origin'][2]}"/>
+          </xacro:if>
+          <xacro:if value="${props_name != 'coxa'}">
+            <origin xyz="${props['link']['origin'][0]}
+                         ${props['link']['origin'][1]}
+                         ${props['link']['origin'][2]}"
+                    rpy="${props['link']['rpy'][0]}
+                         ${props['link']['rpy'][1]}
+                         ${props['link']['rpy'][2]}"/>
+          </xacro:if>
         </visual>
         <collision>
@@ -54,5 +76,7 @@
         <xacro:if value="${not (parent_name == 'base_link')}">
           <parent link="${leg_prefix}_${parent['name']}" />
-          <origin xyz="${child['joint']['origin'][0]}"
+          <origin xyz="${child['joint']['origin'][0]}
+                       ${child['joint']['origin'][1]}
+                       ${child['joint']['origin'][2]}"
                   rpy="0 0 0" />
         </xacro:if>
