Commit message: IMA endin'

File: model/body.urdf.xacro (robot description, xacro)
@@ -8,21 +8,15 @@
       <visual>
         <geometry>
-          <xacro:property name="mesh_file" value="${props['body']['link']['mesh_file']}" />
-          <xacro:if value="${mesh_file == 'None'}">
-            <box size="${props['body']['link']['length']}
-                       ${props['body']['link']['width']}
-                       ${props['body']['link']['thickness']}" />
-          </xacro:if>
-          <xacro:if value="${mesh_file != 'None'}">
-            <mesh filename="${mesh_file}" scale="1 1 1" />
-          </xacro:if>
-          <!-- <material name="${props['body']['link']['material']}"/> -->
+        <xacro:property name="mesh_file" value="${props['body']['link']['mesh_file']}" />
+        <xacro:if value="${mesh_file == 'None'}">
+          <box size="${props['body']['link']['length']}
+                     ${props['body']['link']['width']}
+                     ${props['body']['link']['thickness']}" />
+        </xacro:if>
+        <xacro:if value="${mesh_file != 'None'}">
+          <mesh filename="${mesh_file}" scale="1 1 1" />
+        </xacro:if>
         </geometry>
-        <origin xyz="${props['body']['link']['origin'][0]}
-                     ${props['body']['link']['origin'][1]}
-                     ${props['body']['link']['origin'][2]}"
-                rpy="${props['body']['link']['rpy'][0]}
-                     ${props['body']['link']['rpy'][1]}
-                     ${props['body']['link']['rpy'][2]}"/>
+        <origin xyz="0 0 0" />
       </visual>
       <collision>
@@ -34,15 +28,11 @@
       </collision>
       <inertial>
-        <mass value="${props['body']['inertial']['mass']}" />
-        <inertia ixx="${props['body']['inertial']['inertia']['ixx']}"
-                 ixy="${props['body']['inertial']['inertia']['ixy']}"
-                 ixz="${props['body']['inertial']['inertia']['ixz']}"
-                 iyy="${props['body']['inertial']['inertia']['iyy']}"
-                 iyz="${props['body']['inertial']['inertia']['iyz']}"
-                 izz="${props['body']['inertial']['inertia']['izz']}" />
-         <origin xyz="${props['body']['inertial']['origin'][0]}
-                      ${props['body']['inertial']['origin'][1]}
-                      ${props['body']['inertial']['origin'][2]}"
-                 rpy="0 0 0" />
+        <mass value="${props['body']['inertia']['mass']}" />
+        <inertia ixx="${props['body']['inertia']['inertia']['ixx']}"
+                 ixy="${props['body']['inertia']['inertia']['ixy']}"
+                 ixz="${props['body']['inertia']['inertia']['ixz']}"
+                 iyy="${props['body']['inertia']['inertia']['iyy']}"
+                 iyz="${props['body']['inertia']['inertia']['iyz']}"
+                 izz="${props['body']['inertia']['inertia']['izz']}" />
       </inertial>
     </link>

File: model/leg.urdf.xacro (robot description, xacro)
@@ -8,7 +8,7 @@
     <xacro:if value="${reflect}"> <xacro:property name="reflect_multiplier" value="1" /> </xacro:if>
     <xacro:if value="${not reflect}"> <xacro:property name="reflect_multiplier" value="-1" />   </xacro:if>
-    <xacro:if value="${leg_pos=='rear'}"> <xacro:property name="leg_pos_val" value="${-robot_props['body']['length']/2}" /> </xacro:if>
+    <xacro:if value="${leg_pos=='rear'}"> <xacro:property name="leg_pos_val" value="${-robot_props['body']['link']['length']/2}" /> </xacro:if>
     <xacro:if value="${leg_pos=='central'}"> <xacro:property name="leg_pos_val" value="0" /> </xacro:if>
-    <xacro:if value="${leg_pos=='front'}"> <xacro:property name="leg_pos_val" value="${robot_props['body']['length']/2}" /> </xacro:if>
+    <xacro:if value="${leg_pos=='front'}"> <xacro:property name="leg_pos_val" value="${robot_props['body']['link']['length']/2}" /> </xacro:if>
     <!-- LEG LINK -->
     <xacro:macro name="leg_link" params="props">
@@ -16,9 +16,23 @@
         <visual>
           <geometry>
-            <cylinder length="${props['link']['length']}"
-                      radius="${props['link']['radius']}" />
+            <xacro:property name="mesh_file" value="${props['link']['mesh_file']}" />
+            <xacro:if value="${mesh_file == 'None'}">
+              <cylinder length="${props['link']['length']}"
+                        radius="${props['link']['radius']}" />
+            </xacro:if>
+            <xacro:if value="${mesh_file != 'None'}">
+              <mesh filename="${mesh_file}" scale="1 1 1" />
+            </xacro:if>
           </geometry>
-          <origin xyz="0 0 -${props['link']['length']/2}"
-                  rpy="0 0 ${pi/2}" />
+          <xacro:property name="mesh_file" value="${props['link']['mesh_file']}" />
+          <xacro:if value="${mesh_file == 'None'}">
+            <origin xyz="0 0 -${props['link']['length']/2}"
+                    rpy="0 0 0" />
+          </xacro:if>
+          <xacro:if value="${mesh_file != 'None'}">
+            <mesh filename="${mesh_file}" scale="1 1 1" />
+            <origin xyz="0 0 -${props['link']['length']/2}"
+                    rpy="${pi/2} 0 0" />
+          </xacro:if>
         </visual>
         <collision>
@@ -30,11 +44,11 @@
         </collision>
         <inertial>
-          <mass value="${props['link']['mass']}" />
-          <inertia ixx="${props['link']['inertia']['ixx']}"
-                   ixy="${props['link']['inertia']['ixy']}"
-                   ixz="${props['link']['inertia']['ixz']}"
-                   iyy="${props['link']['inertia']['iyy']}"
-                   iyz="${props['link']['inertia']['iyz']}"
-                   izz="${props['link']['inertia']['izz']}" />
+          <mass value="${props['inertia']['mass']}" />
+          <inertia ixx="${props['inertia']['inertia']['ixx']}"
+                   ixy="${props['inertia']['inertia']['ixy']}"
+                   ixz="${props['inertia']['inertia']['ixz']}"
+                   iyy="${props['inertia']['inertia']['iyy']}"
+                   iyz="${props['inertia']['inertia']['iyz']}"
+                   izz="${props['inertia']['inertia']['izz']}" />
         </inertial>
       </link>
@@ -48,11 +62,12 @@
           <parent link="base_link" />
           <origin xyz="${leg_pos_val}
-                       ${reflect_multiplier*robot_props['body']['width']/2}
+                       ${reflect_multiplier*robot_props['body']['link']['width']/2}
                        0"
-                  rpy="${reflect_multiplier*pi/2} 0 0" />
+                  rpy="${-pi/2} 0 ${reflect_multiplier*pi/2+pi/2}" />
         </xacro:if>
+        <!-- ${reflect_multiplier*pi/2} -->
         <xacro:if value="${not (parent_name == 'base_link')}">
           <parent link="${leg_prefix}_${parent['name']}" />
-          <origin xyz="${child['joint']['origin'][0]}"
+          <origin xyz="${parent['joint']['origin'][0]}"
                   rpy="0 0 0" />
         </xacro:if>
@@ -86,11 +101,11 @@
     <xacro:leg_joint parent="${robot_props['body']}"
                      child="${robot_props['coxa']}"
-                     axis="0 -1 0" />
+                     axis="0 ${reflect_multiplier*1} 0" />
     <xacro:leg_joint parent="${robot_props['coxa']}"
                      child="${robot_props['femur']}"
-                     axis="${reflect_multiplier*1} 0 0" />
+                     axis="1 0 0" />
     <xacro:leg_joint parent="${robot_props['femur']}"
                      child="${robot_props['tibia']}"
-                     axis="${reflect_multiplier*1} 0 0" />
+                     axis="1 0 0" />
   </xacro:macro>
 </robot>
