Commit message: Robot props in YAML

File: robot.urdf (robot description, URDF)
Before this commit: robot the_Walking_thread, 19 links, 18 joints
Links:
- link left_central_coax: geometry collision sphere radius=0.001; visual cylinder length=0.01 radius=0.001
- link left_central_femur: geometry collision sphere radius=0.025; visual cylinder length=0.2 radius=0.025
- link left_central_tibia: geometry collision sphere radius=0.025; visual cylinder length=0.2 radius=0.025
- link left_front_coax: geometry collision sphere radius=0.001; visual cylinder length=0.01 radius=0.001
- link left_front_femur: geometry collision sphere radius=0.025; visual cylinder length=0.2 radius=0.025
- link left_front_tibia: geometry collision sphere radius=0.025; visual cylinder length=0.2 radius=0.025
- link left_rear_coax: geometry collision sphere radius=0.001; visual cylinder length=0.01 radius=0.001
- link left_rear_femur: geometry collision sphere radius=0.025; visual cylinder length=0.2 radius=0.025
- link left_rear_tibia: geometry collision sphere radius=0.025; visual cylinder length=0.2 radius=0.025
- link right_central_coax: geometry collision sphere radius=0.001; visual cylinder length=0.01 radius=0.001
- link right_central_femur: geometry collision sphere radius=0.025; visual cylinder length=0.2 radius=0.025
- link right_central_tibia: geometry collision sphere radius=0.025; visual cylinder length=0.2 radius=0.025
- link right_front_coax: geometry collision sphere radius=0.001; visual cylinder length=0.01 radius=0.001
- link right_front_femur: geometry collision sphere radius=0.025; visual cylinder length=0.2 radius=0.025
- link right_front_tibia: geometry collision sphere radius=0.025; visual cylinder length=0.2 radius=0.025
- link right_rear_coax: geometry collision sphere radius=0.001; visual cylinder length=0.01 radius=0.001
- link right_rear_femur: geometry collision sphere radius=0.025; visual cylinder length=0.2 radius=0.025
- link right_rear_tibia: geometry collision sphere radius=0.025; visual cylinder length=0.2 radius=0.025
Joints:
- removed joint left_central_coax_joint
- removed joint left_central_femur_joint
- removed joint left_central_tibia_joint
- removed joint left_front_coax_joint
- removed joint left_front_femur_joint
- removed joint left_front_tibia_joint
- removed joint left_rear_coax_joint
- removed joint left_rear_femur_joint
- removed joint left_rear_tibia_joint
- removed joint right_central_coax_joint
- removed joint right_central_femur_joint
- removed joint right_central_tibia_joint
- removed joint right_front_coax_joint
- removed joint right_front_femur_joint
- removed joint right_front_tibia_joint
- removed joint right_rear_coax_joint
- removed joint right_rear_femur_joint
- removed joint right_rear_tibia_joint
- added joint left_central_base_link_to_coax_joint: type revolute, parent base_link, child left_central_coax, origin xyz=0                        0.075                        0 rpy=1.57079632679 0 0, axis 0 -1 0, limit lower=-0.785398163397 upper=0.785398163397 effort=0.2 velocity=0.2
- added joint left_central_coax_to_femur_joint: type revolute, parent left_central_coax, child left_central_femur, origin xyz=0 0 -0.01 rpy=0 0 0, axis 1 0 0, limit lower=-0.785398163397 upper=0.785398163397 effort=0.2 velocity=0.2
- added joint left_central_femur_to_tibia_joint: type revolute, parent left_central_femur, child left_central_tibia, origin xyz=0 0 -0.2 rpy=0 0 0, axis 1 0 0, limit lower=-2.35619449019 upper=0.0 effort=0.2 velocity=0.2
- added joint left_front_base_link_to_coax_joint: type revolute, parent base_link, child left_front_coax, origin xyz=0.15                        0.075                        0 rpy=1.57079632679 0 0, axis 0 -1 0, limit lower=-0.785398163397 upper=0.785398163397 effort=0.2 velocity=0.2
- added joint left_front_coax_to_femur_joint: type revolute, parent left_front_coax, child left_front_femur, origin xyz=0 0 -0.01 rpy=0 0 0, axis 1 0 0, limit lower=-0.785398163397 upper=0.785398163397 effort=0.2 velocity=0.2
- added joint left_front_femur_to_tibia_joint: type revolute, parent left_front_femur, child left_front_tibia, origin xyz=0 0 -0.2 rpy=0 0 0, axis 1 0 0, limit lower=-2.35619449019 upper=0.0 effort=0.2 velocity=0.2
- added joint left_rear_base_link_to_coax_joint: type revolute, parent base_link, child left_rear_coax, origin xyz=-0.15                        0.075                        0 rpy=1.57079632679 0 0, axis 0 -1 0, limit lower=-0.785398163397 upper=0.785398163397 effort=0.2 velocity=0.2
- added joint left_rear_coax_to_femur_joint: type revolute, parent left_rear_coax, child left_rear_femur, origin xyz=0 0 -0.01 rpy=0 0 0, axis 1 0 0, limit lower=-0.785398163397 upper=0.785398163397 effort=0.2 velocity=0.2
- added joint left_rear_femur_to_tibia_joint: type revolute, parent left_rear_femur, child left_rear_tibia, origin xyz=0 0 -0.2 rpy=0 0 0, axis 1 0 0, limit lower=-2.35619449019 upper=0.0 effort=0.2 velocity=0.2
- added joint right_central_base_link_to_coax_joint: type revolute, parent base_link, child right_central_coax, origin xyz=0                        -0.075                        0 rpy=-1.57079632679 0 0, axis 0 -1 0, limit lower=-0.785398163397 upper=0.785398163397 effort=0.2 velocity=0.2
- added joint right_central_coax_to_femur_joint: type revolute, parent right_central_coax, child right_central_femur, origin xyz=0 0 -0.01 rpy=0 0 0, axis -1 0 0, limit lower=-0.785398163397 upper=0.785398163397 effort=0.2 velocity=0.2
- added joint right_central_femur_to_tibia_joint: type revolute, parent right_central_femur, child right_central_tibia, origin xyz=0 0 -0.2 rpy=0 0 0, axis -1 0 0, limit lower=-2.35619449019 upper=0.0 effort=0.2 velocity=0.2
- added joint right_front_base_link_to_coax_joint: type revolute, parent base_link, child right_front_coax, origin xyz=0.15                        -0.075                        0 rpy=-1.57079632679 0 0, axis 0 -1 0, limit lower=-0.785398163397 upper=0.785398163397 effort=0.2 velocity=0.2
- added joint right_front_coax_to_femur_joint: type revolute, parent right_front_coax, child right_front_femur, origin xyz=0 0 -0.01 rpy=0 0 0, axis -1 0 0, limit lower=-0.785398163397 upper=0.785398163397 effort=0.2 velocity=0.2
- added joint right_front_femur_to_tibia_joint: type revolute, parent right_front_femur, child right_front_tibia, origin xyz=0 0 -0.2 rpy=0 0 0, axis -1 0 0, limit lower=-2.35619449019 upper=0.0 effort=0.2 velocity=0.2
- added joint right_rear_base_link_to_coax_joint: type revolute, parent base_link, child right_rear_coax, origin xyz=-0.15                        -0.075                        0 rpy=-1.57079632679 0 0, axis 0 -1 0, limit lower=-0.785398163397 upper=0.785398163397 effort=0.2 velocity=0.2
- added joint right_rear_coax_to_femur_joint: type revolute, parent right_rear_coax, child right_rear_femur, origin xyz=0 0 -0.01 rpy=0 0 0, axis -1 0 0, limit lower=-0.785398163397 upper=0.785398163397 effort=0.2 velocity=0.2
- added joint right_rear_femur_to_tibia_joint: type revolute, parent right_rear_femur, child right_rear_tibia, origin xyz=0 0 -0.2 rpy=0 0 0, axis -1 0 0, limit lower=-2.35619449019 upper=0.0 effort=0.2 velocity=0.2

Commit message: The walking thread integration

File: robot.urdf (robot description, URDF)
Before this commit: robot hexapod, 19 links, 18 joints
Links:
- link base_link: mass 0.12138 -> 0.209677; geometry collision box size=0.3618 0.117 0.0525; visual mesh filename=stl/the_walking_thread/frame.stl scale=1 1 1
- link left_central_coxa: mass 0.12138 -> 0.12131; geometry collision sphere radius=0.019; visual mesh filename=stl/the_walking_thread/coxa.stl scale=1 1 1
- link left_central_femur: mass 0.12138 -> 0.02748837
- link left_central_tibia: mass 0.12138 -> 0.08475
- link left_front_coxa: mass 0.12138 -> 0.12131; geometry collision sphere radius=0.019; visual mesh filename=stl/the_walking_thread/coxa.stl scale=1 1 1
- link left_front_femur: mass 0.12138 -> 0.02748837
- link left_front_tibia: mass 0.12138 -> 0.08475
- link left_rear_coxa: mass 0.12138 -> 0.12131; geometry collision sphere radius=0.019; visual mesh filename=stl/the_walking_thread/coxa.stl scale=1 1 1
- link left_rear_femur: mass 0.12138 -> 0.02748837
- link left_rear_tibia: mass 0.12138 -> 0.08475
- link right_central_coxa: mass 0.12138 -> 0.12131; geometry collision sphere radius=0.019; visual mesh filename=stl/the_walking_thread/coxa.stl scale=1 1 1
- link right_central_femur: mass 0.12138 -> 0.02748837
- link right_central_tibia: mass 0.12138 -> 0.08475
- link right_front_coxa: mass 0.12138 -> 0.12131; geometry collision sphere radius=0.019; visual mesh filename=stl/the_walking_thread/coxa.stl scale=1 1 1
- link right_front_femur: mass 0.12138 -> 0.02748837
- link right_front_tibia: mass 0.12138 -> 0.08475
- link right_rear_coxa: mass 0.12138 -> 0.12131; geometry collision sphere radius=0.019; visual mesh filename=stl/the_walking_thread/coxa.stl scale=1 1 1
- link right_rear_femur: mass 0.12138 -> 0.02748837
- link right_rear_tibia: mass 0.12138 -> 0.08475
Joints:
- joint left_central_base_link_to_coxa_joint: origin xyz=0                        0.068                        0 rpy=-1.57079632679 0 3.14159265359 -> xyz=0                        0.0585                        0 rpy=-1.57079632679 0 3.14159265359
- joint left_central_coxa_to_femur_joint: origin xyz=0 -0.01730 -0.036 rpy=0 0 0 -> xyz=0 -0.019 -0.0365 rpy=0 0 0
- joint left_central_femur_to_tibia_joint: origin xyz=0 0 -0.055 rpy=0 0 0 -> xyz=0 0 -0.057 rpy=0 0 0
- joint left_front_base_link_to_coxa_joint: origin xyz=0.1809                        0.068                        0 rpy=-1.57079632679 0 3.14159265359 -> xyz=0.1809                        0.0585                        0 rpy=-1.57079632679 0 3.14159265359
- joint left_front_coxa_to_femur_joint: origin xyz=0 -0.01730 -0.036 rpy=0 0 0 -> xyz=0 -0.019 -0.0365 rpy=0 0 0
- joint left_front_femur_to_tibia_joint: origin xyz=0 0 -0.055 rpy=0 0 0 -> xyz=0 0 -0.057 rpy=0 0 0
- joint left_rear_base_link_to_coxa_joint: origin xyz=-0.1809                        0.068                        0 rpy=-1.57079632679 0 3.14159265359 -> xyz=-0.1809                        0.0585                        0 rpy=-1.57079632679 0 3.14159265359
- joint left_rear_coxa_to_femur_joint: origin xyz=0 -0.01730 -0.036 rpy=0 0 0 -> xyz=0 -0.019 -0.0365 rpy=0 0 0
- joint left_rear_femur_to_tibia_joint: origin xyz=0 0 -0.055 rpy=0 0 0 -> xyz=0 0 -0.057 rpy=0 0 0
- joint right_central_base_link_to_coxa_joint: origin xyz=0                        -0.068                        0 rpy=-1.57079632679 0 0.0 -> xyz=0                        -0.0585                        0 rpy=-1.57079632679 0 0.0
- joint right_central_coxa_to_femur_joint: origin xyz=0 -0.01730 -0.036 rpy=0 0 0 -> xyz=0 -0.019 -0.0365 rpy=0 0 0
- joint right_central_femur_to_tibia_joint: origin xyz=0 0 -0.055 rpy=0 0 0 -> xyz=0 0 -0.057 rpy=0 0 0
- joint right_front_base_link_to_coxa_joint: origin xyz=0.1809                        -0.068                        0 rpy=-1.57079632679 0 0.0 -> xyz=0.1809                        -0.0585                        0 rpy=-1.57079632679 0 0.0
- joint right_front_coxa_to_femur_joint: origin xyz=0 -0.01730 -0.036 rpy=0 0 0 -> xyz=0 -0.019 -0.0365 rpy=0 0 0
- joint right_front_femur_to_tibia_joint: origin xyz=0 0 -0.055 rpy=0 0 0 -> xyz=0 0 -0.057 rpy=0 0 0
- joint right_rear_base_link_to_coxa_joint: origin xyz=-0.1809                        -0.068                        0 rpy=-1.57079632679 0 0.0 -> xyz=-0.1809                        -0.0585                        0 rpy=-1.57079632679 0 0.0
- joint right_rear_coxa_to_femur_joint: origin xyz=0 -0.01730 -0.036 rpy=0 0 0 -> xyz=0 -0.019 -0.0365 rpy=0 0 0
- joint right_rear_femur_to_tibia_joint: origin xyz=0 0 -0.055 rpy=0 0 0 -> xyz=0 0 -0.057 rpy=0 0 0
