Commit message: Props as argument

File: hexapod.urdf.xacro (robot description, xacro)
@@ -1,14 +1,15 @@
 <?xml version="1.0" encoding="utf-8"?>
-<robot name="the_Walking_thread" xmlns:xacro="http://www.ros.org/wiki/xacro">
+<robot name="hexapod" xmlns:xacro="http://www.ros.org/wiki/xacro">
+  <xacro:arg name="props_path" default="$(cwd)/config/props.yaml" />
   <!-- BODY DEFINITION -->
-  <xacro:include filename="$(cwd)/model/body.urdf.xacro" ns="macros"/>
-  <xacro:macros.body/>
+  <xacro:include filename="$(cwd)/model/body.urdf.xacro" ns="body" />
+  <xacro:body.body props_path="$(arg props_path)" />
   <!-- LED DEFINITION -->
-  <xacro:include filename="$(cwd)/model/leg.urdf.xacro" ns="macros"/>
-  <xacro:macros.leg leg_prefix="left_front" reflect="true" leg_number="front"/>
-  <xacro:macros.leg leg_prefix="left_central" reflect="true" leg_number="central"/>
-  <xacro:macros.leg leg_prefix="left_rear" reflect="true" leg_number="rear"/>
-  <xacro:macros.leg leg_prefix="right_front" reflect="false" leg_number="front"/>
-  <xacro:macros.leg leg_prefix="right_central" reflect="false" leg_number="central"/>
-  <xacro:macros.leg leg_prefix="right_rear" reflect="false" leg_number="rear"/>
+  <xacro:include filename="$(cwd)/model/leg.urdf.xacro" ns="leg" />
+  <xacro:leg.leg leg_prefix="left_front" reflect="true" leg_number="front" props_path="$(arg props_path)" />
+  <xacro:leg.leg leg_prefix="left_central" reflect="true" leg_number="central" props_path="$(arg props_path)" />
+  <xacro:leg.leg leg_prefix="left_rear" reflect="true" leg_number="rear" props_path="$(arg props_path)" />
+  <xacro:leg.leg leg_prefix="right_front" reflect="false" leg_number="front" props_path="$(arg props_path)" />
+  <xacro:leg.leg leg_prefix="right_central" reflect="false" leg_number="central" props_path="$(arg props_path)" />
+  <xacro:leg.leg leg_prefix="right_rear" reflect="false" leg_number="rear" props_path="$(arg props_path)" />
 </robot>

File: model/body.urdf.xacro (robot description, xacro)
@@ -2,21 +2,21 @@
 <robot xmlns:xacro="http://www.ros.org/wiki/xacro">
   <!-- body defining macro -->
-  <xacro:macro name="body">
-    <xacro:property name="yaml_file" value="$(cwd)/config/props.yaml" />
-    <xacro:property name="props" value="${load_yaml(yaml_file)}"/>
+  <xacro:macro name="body" params="props_path">
+    <xacro:property name="yaml_file" value="${props_path}"  />
+    <xacro:property name="props" value="${load_yaml(yaml_file)}" />
     <link name="${props['body']['name']}">
       <visual>
         <geometry>
-          <box size="${props['body']['length']} ${props['body']['width']} ${props['body']['thickness']}"/>
+          <box size="${props['body']['length']} ${props['body']['width']} ${props['body']['thickness']}" />
         </geometry>
-        <origin xyz="0 0 0"/>
+        <origin xyz="0 0 0" />
       </visual>
       <collision>
         <geometry>
-          <box size="${props['body']['length']} ${props['body']['width']} ${props['body']['thickness']}"/>
+          <box size="${props['body']['length']} ${props['body']['width']} ${props['body']['thickness']}" />
         </geometry>
       </collision>
       <inertial>
-        <mass value="${props['body']['mass']}"/>
+        <mass value="${props['body']['mass']}" />
         <inertia ixx="${props['body']['inertia']['ixx']}"
                  ixy="${props['body']['inertia']['ixy']}"
@@ -24,5 +24,5 @@
                  iyy="${props['body']['inertia']['iyy']}"
                  iyz="${props['body']['inertia']['iyz']}"
-                 izz="${props['body']['inertia']['izz']}"/>
+                 izz="${props['body']['inertia']['izz']}" />
       </inertial>
     </link>

File: model/leg.urdf.xacro (robot description, xacro)
@@ -2,22 +2,22 @@
 <robot xmlns:xacro="http://www.ros.org/wiki/xacro">
   <!-- LEG MACRO -->
-  <xacro:macro name="leg" params="leg_prefix reflect leg_number">
-    <xacro:property name="yaml_file" value="$(cwd)/config/props.yaml"/>
-    <xacro:property name="robot_props" value="${load_yaml(yaml_file)}"/>
+  <xacro:macro name="leg" params="leg_prefix reflect leg_number props_path">
+    <xacro:property name="yaml_file" value="${props_path}" />
+    <xacro:property name="robot_props" value="${load_yaml(yaml_file)}" />
     <!-- coditional blocks -->
     <xacro:if value="${reflect}">
-      <xacro:property name="reflect_multiplier" value="1" scope="parent"/>
+      <xacro:property name="reflect_multiplier" value="1" scope="parent" />
     </xacro:if>
     <xacro:if value="${not reflect}">
-      <xacro:property name="reflect_multiplier" value="-1" scope="parent"/>
+      <xacro:property name="reflect_multiplier" value="-1" scope="parent" />
     </xacro:if>
     <xacro:if value="${leg_number == 'rear'}">
-      <xacro:property name="leg_pos" value="${-robot_props['body']['length']/2}" scope="parent"/>
+      <xacro:property name="leg_pos" value="${-robot_props['body']['length']/2}" scope="parent" />
     </xacro:if>
     <xacro:if value="${leg_number == 'central'}">
-      <xacro:property name="leg_pos" value="0" scope="parent"/>
+      <xacro:property name="leg_pos" value="0" scope="parent" />
     </xacro:if>
     <xacro:if value="${leg_number == 'front'}">
-      <xacro:property name="leg_pos" value="${robot_props['body']['length']/2}" scope="parent"/>
+      <xacro:property name="leg_pos" value="${robot_props['body']['length']/2}" scope="parent" />
     </xacro:if>
     <!-- LEG LINK -->
@@ -27,18 +27,18 @@
           <geometry>
             <cylinder length="${props['link']['length']}"
-                      radius="${props['link']['radius']}"/>
+                      radius="${props['link']['radius']}" />
           </geometry>
           <origin xyz="0 0 -${props['link']['length']/2}"
-                  rpy="0 0 ${pi/2}"/>
+                  rpy="0 0 ${pi/2}" />
         </visual>
         <collision>
           <geometry>
-            <sphere radius="${props['link']['radius']}"/>
+            <sphere radius="${props['link']['radius']}" />
           </geometry>
           <origin xyz="0 0 -${(props['link']['length']-(props['link']['radius']/2))}"
-                  rpy="0 0 0"/>
+                  rpy="0 0 0" />
         </collision>
         <inertial>
-          <mass value="${props['link']['mass']}"/>
+          <mass value="${props['link']['mass']}" />
           <inertia ixx="${props['link']['inertia']['ixx']}"
                    ixy="${props['link']['inertia']['ixy']}"
@@ -46,5 +46,5 @@
                    iyy="${props['link']['inertia']['iyy']}"
                    iyz="${props['link']['inertia']['iyz']}"
-                   izz="${props['link']['inertia']['izz']}"/>
+                   izz="${props['link']['inertia']['izz']}" />
         </inertial>
       </link>
@@ -54,41 +54,41 @@
       <joint name="${leg_prefix}_${parent['name']}_to_${child['name']}_joint"
              type="revolute">
-        <xacro:property name="parent_name" value="${parent['name']}"/>
+        <xacro:property name="parent_name" value="${parent['name']}" />
         <xacro:if value="${parent_name == 'base_link'}">
-          <parent link="base_link"/>
+          <parent link="base_link" />
           <origin xyz="${leg_pos}
                        ${reflect_multiplier*robot_props['body']['width']/2}
                        0"
-                  rpy="${reflect_multiplier*pi/2} 0 0"/>
+                  rpy="${reflect_multiplier*pi/2} 0 0" />
         </xacro:if>
         <xacro:if value="${not (parent_name == 'base_link')}">
-          <parent link="${leg_prefix}_${parent['name']}"/>
+          <parent link="${leg_prefix}_${parent['name']}" />
           <origin xyz="${child['joint']['origin'][0]}"
-                  rpy="0 0 0"/>
+                  rpy="0 0 0" />
         </xacro:if>
-        <child link="${leg_prefix}_${child['name']}"/>
-        <axis xyz="${axis}"/>
-        <xacro:property name="low_lim" value="${child['joint']['limit']['lower']}"/>
-        <xacro:property name="up_lim" value="${child['joint']['limit']['upper']}"/>
+        <child link="${leg_prefix}_${child['name']}" />
+        <axis xyz="${axis}" />
+        <xacro:property name="low_lim" value="${child['joint']['limit']['lower']}" />
+        <xacro:property name="up_lim" value="${child['joint']['limit']['upper']}" />
         <limit effort="${robot_props['servo']['effort']}"
                lower="${radians(low_lim)}"
                upper="${radians(up_lim)}"
-               velocity="${robot_props['servo']['velocity']}"/>
+               velocity="${robot_props['servo']['velocity']}" />
       </joint>
     </xacro:macro>
     <!-- DEFINE LINKS -->
-    <xacro:leg_link props="${robot_props['coxa']}"/>
-    <xacro:leg_link props="${robot_props['femur']}"/>
-    <xacro:leg_link props="${robot_props['tibia']}"/>
+    <xacro:leg_link props="${robot_props['coxa']}" />
+    <xacro:leg_link props="${robot_props['femur']}" />
+    <xacro:leg_link props="${robot_props['tibia']}" />
     <!-- DEFINE JOINTS -->
     <xacro:leg_joint parent="${robot_props['body']}"
                      child="${robot_props['coxa']}"
-                     axis="0 -1 0"/>
+                     axis="0 -1 0" />
     <xacro:leg_joint parent="${robot_props['coxa']}"
                      child="${robot_props['femur']}"
-                     axis="${reflect_multiplier*1} 0 0"/>
+                     axis="${reflect_multiplier*1} 0 0" />
     <xacro:leg_joint parent="${robot_props['femur']}"
                      child="${robot_props['tibia']}"
-                     axis="${reflect_multiplier*1} 0 0"/>
+                     axis="${reflect_multiplier*1} 0 0" />
   </xacro:macro>
 </robot>

File: robot.urdf (robot description, URDF)
Before this commit: robot the_Walking_thread, 19 links, 18 joints
Links:
- removed link left_central_coax
- removed link left_front_coax
- removed link left_rear_coax
- removed link right_central_coax
- removed link right_front_coax
- removed link right_rear_coax
- added link left_central_coxa, mass 0.2; collision sphere radius=0.001; visual cylinder length=0.01 radius=0.001
- added link left_front_coxa, mass 0.2; collision sphere radius=0.001; visual cylinder length=0.01 radius=0.001
- added link left_rear_coxa, mass 0.2; collision sphere radius=0.001; visual cylinder length=0.01 radius=0.001
- added link right_central_coxa, mass 0.2; collision sphere radius=0.001; visual cylinder length=0.01 radius=0.001
- added link right_front_coxa, mass 0.2; collision sphere radius=0.001; visual cylinder length=0.01 radius=0.001
- added link right_rear_coxa, mass 0.2; collision sphere radius=0.001; visual cylinder length=0.01 radius=0.001
Joints:
- removed joint left_central_base_link_to_coax_joint
- removed joint left_central_coax_to_femur_joint
- removed joint left_front_base_link_to_coax_joint
- removed joint left_front_coax_to_femur_joint
- removed joint left_rear_base_link_to_coax_joint
- removed joint left_rear_coax_to_femur_joint
- removed joint right_central_base_link_to_coax_joint
- removed joint right_central_coax_to_femur_joint
- removed joint right_front_base_link_to_coax_joint
- removed joint right_front_coax_to_femur_joint
- removed joint right_rear_base_link_to_coax_joint
- removed joint right_rear_coax_to_femur_joint
- added joint left_central_base_link_to_coxa_joint: type revolute, parent base_link, child left_central_coxa, origin xyz=0                        0.075                        0 rpy=1.57079632679 0 0, axis 0 -1 0, limit lower=-0.785398163397 upper=0.785398163397 effort=0.2 velocity=0.2
- added joint left_central_coxa_to_femur_joint: type revolute, parent left_central_coxa, child left_central_femur, origin xyz=0 0 -0.01 rpy=0 0 0, axis 1 0 0, limit lower=-0.785398163397 upper=0.785398163397 effort=0.2 velocity=0.2
- added joint left_front_base_link_to_coxa_joint: type revolute, parent base_link, child left_front_coxa, origin xyz=0.15                        0.075                        0 rpy=1.57079632679 0 0, axis 0 -1 0, limit lower=-0.785398163397 upper=0.785398163397 effort=0.2 velocity=0.2
- added joint left_front_coxa_to_femur_joint: type revolute, parent left_front_coxa, child left_front_femur, origin xyz=0 0 -0.01 rpy=0 0 0, axis 1 0 0, limit lower=-0.785398163397 upper=0.785398163397 effort=0.2 velocity=0.2
- added joint left_rear_base_link_to_coxa_joint: type revolute, parent base_link, child left_rear_coxa, origin xyz=-0.15                        0.075                        0 rpy=1.57079632679 0 0, axis 0 -1 0, limit lower=-0.785398163397 upper=0.785398163397 effort=0.2 velocity=0.2
- added joint left_rear_coxa_to_femur_joint: type revolute, parent left_rear_coxa, child left_rear_femur, origin xyz=0 0 -0.01 rpy=0 0 0, axis 1 0 0, limit lower=-0.785398163397 upper=0.785398163397 effort=0.2 velocity=0.2
- added joint right_central_base_link_to_coxa_joint: type revolute, parent base_link, child right_central_coxa, origin xyz=0                        -0.075                        0 rpy=-1.57079632679 0 0, axis 0 -1 0, limit lower=-0.785398163397 upper=0.785398163397 effort=0.2 velocity=0.2
- added joint right_central_coxa_to_femur_joint: type revolute, parent right_central_coxa, child right_central_femur, origin xyz=0 0 -0.01 rpy=0 0 0, axis -1 0 0, limit lower=-0.785398163397 upper=0.785398163397 effort=0.2 velocity=0.2
- added joint right_front_base_link_to_coxa_joint: type revolute, parent base_link, child right_front_coxa, origin xyz=0.15                        -0.075                        0 rpy=-1.57079632679 0 0, axis 0 -1 0, limit lower=-0.785398163397 upper=0.785398163397 effort=0.2 velocity=0.2
- added joint right_front_coxa_to_femur_joint: type revolute, parent right_front_coxa, child right_front_femur, origin xyz=0 0 -0.01 rpy=0 0 0, axis -1 0 0, limit lower=-0.785398163397 upper=0.785398163397 effort=0.2 velocity=0.2
- added joint right_rear_base_link_to_coxa_joint: type revolute, parent base_link, child right_rear_coxa, origin xyz=-0.15                        -0.075                        0 rpy=-1.57079632679 0 0, axis 0 -1 0, limit lower=-0.785398163397 upper=0.785398163397 effort=0.2 velocity=0.2
- added joint right_rear_coxa_to_femur_joint: type revolute, parent right_rear_coxa, child right_rear_femur, origin xyz=0 0 -0.01 rpy=0 0 0, axis -1 0 0, limit lower=-0.785398163397 upper=0.785398163397 effort=0.2 velocity=0.2

Commit message: Rename variables

File: hexapod.urdf.xacro (robot description, xacro)
@@ -2,14 +2,14 @@
 <robot name="hexapod" xmlns:xacro="http://www.ros.org/wiki/xacro">
   <xacro:arg name="props_path" default="$(cwd)/config/props.yaml" />
-  <!-- BODY DEFINITION -->
+  <!-- BODY DECLARATION -->
   <xacro:include filename="$(cwd)/model/body.urdf.xacro" ns="body" />
   <xacro:body.body props_path="$(arg props_path)" />
-  <!-- LED DEFINITION -->
+  <!-- LED DECLARATION -->
   <xacro:include filename="$(cwd)/model/leg.urdf.xacro" ns="leg" />
-  <xacro:leg.leg leg_prefix="left_front" reflect="true" leg_number="front" props_path="$(arg props_path)" />
-  <xacro:leg.leg leg_prefix="left_central" reflect="true" leg_number="central" props_path="$(arg props_path)" />
-  <xacro:leg.leg leg_prefix="left_rear" reflect="true" leg_number="rear" props_path="$(arg props_path)" />
-  <xacro:leg.leg leg_prefix="right_front" reflect="false" leg_number="front" props_path="$(arg props_path)" />
-  <xacro:leg.leg leg_prefix="right_central" reflect="false" leg_number="central" props_path="$(arg props_path)" />
-  <xacro:leg.leg leg_prefix="right_rear" reflect="false" leg_number="rear" props_path="$(arg props_path)" />
+  <xacro:leg.leg leg_prefix="left_front" reflect="true" leg_pos="front" props_path="$(arg props_path)" />
+  <xacro:leg.leg leg_prefix="left_central" reflect="true" leg_pos="central" props_path="$(arg props_path)" />
+  <xacro:leg.leg leg_prefix="left_rear" reflect="true" leg_pos="rear" props_path="$(arg props_path)" />
+  <xacro:leg.leg leg_prefix="right_front" reflect="false" leg_pos="front" props_path="$(arg props_path)" />
+  <xacro:leg.leg leg_prefix="right_central" reflect="false" leg_pos="central" props_path="$(arg props_path)" />
+  <xacro:leg.leg leg_prefix="right_rear" reflect="false" leg_pos="rear" props_path="$(arg props_path)" />
 </robot>

File: model/leg.urdf.xacro (robot description, xacro)
@@ -2,5 +2,5 @@
 <robot xmlns:xacro="http://www.ros.org/wiki/xacro">
   <!-- LEG MACRO -->
-  <xacro:macro name="leg" params="leg_prefix reflect leg_number props_path">
+  <xacro:macro name="leg" params="leg_prefix reflect leg_pos props_path">
     <xacro:property name="yaml_file" value="${props_path}" />
     <xacro:property name="robot_props" value="${load_yaml(yaml_file)}" />
@@ -12,11 +12,11 @@
       <xacro:property name="reflect_multiplier" value="-1" scope="parent" />
     </xacro:if>
-    <xacro:if value="${leg_number == 'rear'}">
+    <xacro:if value="${leg_pos == 'rear'}">
       <xacro:property name="leg_pos" value="${-robot_props['body']['length']/2}" scope="parent" />
     </xacro:if>
-    <xacro:if value="${leg_number == 'central'}">
+    <xacro:if value="${leg_pos == 'central'}">
       <xacro:property name="leg_pos" value="0" scope="parent" />
     </xacro:if>
-    <xacro:if value="${leg_number == 'front'}">
+    <xacro:if value="${leg_pos == 'front'}">
       <xacro:property name="leg_pos" value="${robot_props['body']['length']/2}" scope="parent" />
     </xacro:if>
