Commit message: integraton with gazebo

File: hexapod.urdf.xacro (robot description, xacro)
@@ -1,19 +1,27 @@
 <?xml version="1.0" encoding="utf-8"?>
 <robot name="hexapod" xmlns:xacro="http://www.ros.org/wiki/xacro">
-  <xacro:arg name="props_path" default="$(cwd)/config/props.yaml" />
+  <xacro:arg name="props_path" default="$(cwd)/config/props/props.yaml" />
+  <xacro:arg name="use_package_relative" default="True" />
+  <xacro:property name="_use_package_relative" value="$(arg use_package_relative)" />
+  <xacro:if value="${_use_package_relative}">
+    <xacro:include filename="$(find the_walking_thread_gazebo)/src/urdf/model/body.urdf.xacro" ns="body" />
+    <xacro:include filename="$(find the_walking_thread_gazebo)/src/urdf/model/leg.urdf.xacro" ns="leg" />
+  </xacro:if>
+  <xacro:unless value="${_use_package_relative}">
+    <xacro:include filename="$(cwd)/model/body.urdf.xacro" ns="body" />
+    <xacro:include filename="$(cwd)/model/leg.urdf.xacro" ns="leg" />
+  </xacro:unless>
   <!-- BODY DECLARATION -->
-  <xacro:include filename="$(cwd)/model/body.urdf.xacro" ns="body" />
-  <xacro:body.body props_path="$(arg props_path)" />
+  <xacro:body.body props_path="$(arg props_path)" use_package_relative="$(arg use_package_relative)" />
   <!-- LED DECLARATION -->
-  <xacro:include filename="$(cwd)/model/leg.urdf.xacro" ns="leg" />
-  <xacro:leg.leg leg_prefix="left_front" reflect="true" leg_pos="front" props_path="$(arg props_path)" />
-  <xacro:leg.leg leg_prefix="left_central" reflect="true" leg_pos="central" props_path="$(arg props_path)" />
-  <xacro:leg.leg leg_prefix="left_rear" reflect="true" leg_pos="rear" props_path="$(arg props_path)" />
-  <xacro:leg.leg leg_prefix="right_front" reflect="false" leg_pos="front" props_path="$(arg props_path)" />
-  <xacro:leg.leg leg_prefix="right_central" reflect="false" leg_pos="central" props_path="$(arg props_path)" />
-  <xacro:leg.leg leg_prefix="right_rear" reflect="false" leg_pos="rear" props_path="$(arg props_path)" />
+  <xacro:leg.leg leg_prefix="left_front" reflect="true" leg_pos="front" props_path="$(arg props_path)" use_package_relative="$(arg use_package_relative)" />
+  <xacro:leg.leg leg_prefix="left_central" reflect="true" leg_pos="central" props_path="$(arg props_path)" use_package_relative="$(arg use_package_relative)" />
+  <xacro:leg.leg leg_prefix="left_rear" reflect="true" leg_pos="rear" props_path="$(arg props_path)" use_package_relative="$(arg use_package_relative)" />
+  <xacro:leg.leg leg_prefix="right_front" reflect="false" leg_pos="front" props_path="$(arg props_path)" use_package_relative="$(arg use_package_relative)" />
+  <xacro:leg.leg leg_prefix="right_central" reflect="false" leg_pos="central" props_path="$(arg props_path)" use_package_relative="$(arg use_package_relative)" />
+  <xacro:leg.leg leg_prefix="right_rear" reflect="false" leg_pos="rear" props_path="$(arg props_path)" use_package_relative="$(arg use_package_relative)" />
   <gazebo>
     <plugin name="gazebo_ros_control" filename="libgazebo_ros_control.so">
-      <robotNamespace>/</robotNamespace>
+      <robotNamespace>/simple_model</robotNamespace>
     </plugin>
   </gazebo>

File: model/body.urdf.xacro (robot description, xacro)
@@ -2,5 +2,5 @@
 <robot xmlns:xacro="http://www.ros.org/wiki/xacro">
   <!-- body defining macro -->
-  <xacro:macro name="body" params="props_path">
+  <xacro:macro name="body" params="props_path use_package_relative">
     <xacro:property name="yaml_file" value="${props_path}"  />
     <xacro:property name="props" value="${load_yaml(yaml_file)}" />
@@ -14,7 +14,12 @@
                      ${props['body']['link']['thickness']}" />
         </xacro:if>
-        <xacro:if value="${mesh_file != 'None'}">
-          <mesh filename="${mesh_file}" scale="1 1 1" />
-        </xacro:if>
+        <xacro:unless value="${mesh_file == 'None'}">
+          <xacro:if value="${use_package_relative}">
+            <mesh filename="package://${props['package']['name']}/${props['package']['meshes_path']}/${mesh_file}" scale="1 1 1" />
+          </xacro:if>
+          <xacro:unless value="${use_package_relative}">
+            <mesh filename="${mesh_file}" scale="1 1 1" />
+          </xacro:unless>
+        </xacro:unless>
         </geometry>
         <origin xyz="0 0 0" />

File: model/leg.urdf.xacro (robot description, xacro)
@@ -2,13 +2,13 @@
 <robot xmlns:xacro="http://www.ros.org/wiki/xacro">
   <!-- LEG MACRO -->
-  <xacro:macro name="leg" params="leg_prefix reflect leg_pos props_path">
+  <xacro:macro name="leg" params="leg_prefix reflect leg_pos props_path use_package_relative">
     <xacro:property name="yaml_file" value="${props_path}" />
     <xacro:property name="robot_props" value="${load_yaml(yaml_file)}" />
     <!-- CONDITIONAL BLOCKS -->
     <xacro:if value="${reflect}"> <xacro:property name="reflect_multiplier" value="1" /> </xacro:if>
-    <xacro:if value="${not reflect}"> <xacro:property name="reflect_multiplier" value="-1" />   </xacro:if>
-    <xacro:if value="${leg_pos=='rear'}"> <xacro:property name="leg_pos_val" value="${-robot_props['body']['link']['length']/2}" /> </xacro:if>
-    <xacro:if value="${leg_pos=='central'}"> <xacro:property name="leg_pos_val" value="0" /> </xacro:if>
-    <xacro:if value="${leg_pos=='front'}"> <xacro:property name="leg_pos_val" value="${robot_props['body']['link']['length']/2}" /> </xacro:if>
+    <xacro:unless value="${reflect}"> <xacro:property name="reflect_multiplier" value="-1" />   </xacro:unless>
+    <xacro:if value="${leg_pos == 'rear'}"> <xacro:property name="leg_pos_val" value="${-robot_props['body']['link']['length']/2}" /> </xacro:if>
+    <xacro:if value="${leg_pos == 'central'}"> <xacro:property name="leg_pos_val" value="0" /> </xacro:if>
+    <xacro:if value="${leg_pos == 'front'}"> <xacro:property name="leg_pos_val" value="${robot_props['body']['link']['length']/2}" /> </xacro:if>
     <!-- LEG LINK -->
     <xacro:macro name="leg_link" params="props">
@@ -21,7 +21,12 @@
                         radius="${props['link']['radius']}" />
             </xacro:if>
-            <xacro:if value="${mesh_file != 'None'}">
-              <mesh filename="${mesh_file}" scale="1 1 1" />
-            </xacro:if>
+            <xacro:unless value="${mesh_file == 'None'}">
+              <xacro:if value="${use_package_relative}">
+                <mesh filename="package://${robot_props['package']['name']}/${robot_props['package']['meshes_path']}/${mesh_file}" scale="1 1 1" />
+              </xacro:if>
+              <xacro:unless value="${use_package_relative}">
+                <mesh filename="${mesh_file}" scale="1 1 1" />
+              </xacro:unless>
+            </xacro:unless>
           </geometry>
           <xacro:property name="mesh_file" value="${props['link']['mesh_file']}" />
@@ -30,9 +35,8 @@
                     rpy="0 0 0" />
           </xacro:if>
-          <xacro:if value="${mesh_file != 'None'}">
-            <mesh filename="${mesh_file}" scale="1 1 1" />
+          <xacro:unless value="${mesh_file == 'None'}">
             <origin xyz="0 0 -${props['link']['length']/2}"
                     rpy="${pi/2} 0 0" />
-          </xacro:if>
+          </xacro:unless>
         </visual>
         <collision>
@@ -40,5 +44,5 @@
             <sphere radius="${props['link']['radius']}" />
           </geometry>
-          <origin xyz="0 0 -${(props['link']['length']-(props['link']['radius']/2))}"
+          <origin xyz="0 0 -${(props['link']['length']-(props['link']['radius']))}"
                   rpy="0 0 0" />
         </collision>
@@ -66,5 +70,4 @@
                   rpy="${-pi/2} 0 ${reflect_multiplier*pi/2+pi/2}" />
         </xacro:if>
-        <!-- ${reflect_multiplier*pi/2} -->
         <xacro:if value="${not (parent_name == 'base_link')}">
           <parent link="${leg_prefix}_${parent['name']}" />
@@ -82,12 +85,11 @@
       </joint>
       <!-- TRANSMITION DEFINITION -->
-      <transmission name="${leg_prefix}_${parent['name']}_to_${child['name']}_transmition"
-                    type="SimpleTransmission">
+      <transmission name="${leg_prefix}_${parent['name']}_to_${child['name']}_transmition">
         <type>transmission_interface/SimpleTransmission</type>
         <joint name="${leg_prefix}_${parent['name']}_to_${child['name']}_joint">
-          <hardwareInterface>EffortJointInterface</hardwareInterface>
+          <hardwareInterface>hardware_interface/EffortJointInterface</hardwareInterface>
         </joint>
         <actuator name="${leg_prefix}_${parent['name']}_to_${child['name']}_actuator">
-          <hardwareInterface>EffortJointInterface</hardwareInterface>
+          <hardwareInterface>hardware_interface/EffortJointInterface</hardwareInterface>
           <mechanicalReduction>1</mechanicalReduction>
         </actuator>

File: robot.urdf (robot description, URDF)
Before this commit: robot hexapod, 19 links, 18 joints
Links:
- link base_link: geometry collision box size=0.3618 0.117 0.0525; visual mesh filename=meshes/the_walking_thread/frame.stl scale=1 1 1
- link left_central_coxa: geometry collision sphere radius=0.019; visual mesh filename=meshes/the_walking_thread/coxa.stl scale=1 1 1
- link left_central_femur: geometry collision sphere radius=0.03; visual mesh filename=meshes/the_walking_thread/femur.stl scale=1 1 1
- link left_central_tibia: geometry collision sphere radius=0.0065; visual mesh filename=meshes/the_walking_thread/tibia.stl scale=1 1 1
- link left_front_coxa: geometry collision sphere radius=0.019; visual mesh filename=meshes/the_walking_thread/coxa.stl scale=1 1 1
- link left_front_femur: geometry collision sphere radius=0.03; visual mesh filename=meshes/the_walking_thread/femur.stl scale=1 1 1
- link left_front_tibia: geometry collision sphere radius=0.0065; visual mesh filename=meshes/the_walking_thread/tibia.stl scale=1 1 1
- link left_rear_coxa: geometry collision sphere radius=0.019; visual mesh filename=meshes/the_walking_thread/coxa.stl scale=1 1 1
- link left_rear_femur: geometry collision sphere radius=0.03; visual mesh filename=meshes/the_walking_thread/femur.stl scale=1 1 1
- link left_rear_tibia: geometry collision sphere radius=0.0065; visual mesh filename=meshes/the_walking_thread/tibia.stl scale=1 1 1
- link right_central_coxa: geometry collision sphere radius=0.019; visual mesh filename=meshes/the_walking_thread/coxa.stl scale=1 1 1
- link right_central_femur: geometry collision sphere radius=0.03; visual mesh filename=meshes/the_walking_thread/femur.stl scale=1 1 1
- link right_central_tibia: geometry collision sphere radius=0.0065; visual mesh filename=meshes/the_walking_thread/tibia.stl scale=1 1 1
- link right_front_coxa: geometry collision sphere radius=0.019; visual mesh filename=meshes/the_walking_thread/coxa.stl scale=1 1 1
- link right_front_femur: geometry collision sphere radius=0.03; visual mesh filename=meshes/the_walking_thread/femur.stl scale=1 1 1
- link right_front_tibia: geometry collision sphere radius=0.0065; visual mesh filename=meshes/the_walking_thread/tibia.stl scale=1 1 1
- link right_rear_coxa: geometry collision sphere radius=0.019; visual mesh filename=meshes/the_walking_thread/coxa.stl scale=1 1 1
- link right_rear_femur: geometry collision sphere radius=0.03; visual mesh filename=meshes/the_walking_thread/femur.stl scale=1 1 1
- link right_rear_tibia: geometry collision sphere radius=0.0065; visual mesh filename=meshes/the_walking_thread/tibia.stl scale=1 1 1

Commit message: Relative paths

File: hexapod.urdf.xacro (robot description, xacro)
@@ -1,5 +1,5 @@
 <?xml version="1.0" encoding="utf-8"?>
 <robot name="hexapod" xmlns:xacro="http://www.ros.org/wiki/xacro">
-  <xacro:arg name="props_path" default="$(cwd)/config/props/props.yaml" />
+  <xacro:arg name="props_path" default="$(cwd)/config/props/twt_props.yaml" />
   <xacro:arg name="use_package_relative" default="True" />
   <xacro:property name="_use_package_relative" value="$(arg use_package_relative)" />
@@ -23,6 +23,9 @@
   <gazebo>
     <plugin name="gazebo_ros_control" filename="libgazebo_ros_control.so">
-      <robotNamespace>/simple_model</robotNamespace>
+      <robotNamespace>/twt</robotNamespace>
     </plugin>
   </gazebo>
+  <gazebo reference="base_link">
+    <gravity>0</gravity>
+  </gazebo>
 </robot>

File: model/body.urdf.xacro (robot description, xacro)
@@ -3,4 +3,5 @@
   <!-- body defining macro -->
   <xacro:macro name="body" params="props_path use_package_relative">
+    <link name="base_link"></link>
     <xacro:property name="yaml_file" value="${props_path}"  />
     <xacro:property name="props" value="${load_yaml(yaml_file)}" />
@@ -42,4 +43,9 @@
       </inertial>
     </link>
+    <joint name="base_link_to_body_joint" type="fixed">
+      <origin xyz="0 0 0" rpy="0 0 0"/>
+      <parent link="base_link"/>
+      <child link="${props['body']['name']}"/>
+    </joint>
   </xacro:macro>
 </robot>

File: model/leg.urdf.xacro (robot description, xacro)
@@ -63,6 +63,7 @@
              type="revolute">
         <xacro:property name="parent_name" value="${parent['name']}" />
-        <xacro:if value="${parent_name == 'base_link'}">
-          <parent link="base_link" />
+        <xacro:property name="body_link_name" value="${robot_props['body']['name']}" />
+        <xacro:if value="${parent_name == body_link_name}">
+          <parent link="${body_link_name}" />
           <origin xyz="${leg_pos_val}
                        ${reflect_multiplier*robot_props['body']['link']['width']/2}
@@ -70,5 +71,5 @@
                   rpy="${-pi/2} 0 ${reflect_multiplier*pi/2+pi/2}" />
         </xacro:if>
-        <xacro:if value="${not (parent_name == 'base_link')}">
+        <xacro:if value="${not (parent_name == body_link_name)}">
           <parent link="${leg_prefix}_${parent['name']}" />
           <origin xyz="${parent['joint']['origin'][0]}"
@@ -110,4 +111,8 @@
                      child="${robot_props['tibia']}"
                      axis="1 0 0" />
+    <gazebo reference="${leg_prefix}_${robot_props['coxa']['name']}">
+      <mu1>0.9</mu1>
+      <mu2>0.6</mu2>
+    </gazebo>
   </xacro:macro>
 </robot>

File: robot.urdf (robot description, URDF)
Before this commit: robot hexapod, 19 links, 18 joints
Links:
- added link body, mass 0.209677; collision box size=0.3618 0.117 0.0525; visual mesh filename=package://the_walking_thread_gazebo/src/urdf/meshes/the_wal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 scale=1 1 1
- link base_link: mass 0.209677 -> None; geometry 
- link left_central_coxa: geometry collision sphere radius=0.019; visual mesh filename=package://the_walking_thread_gazebo/src/urdf/meshes/the_wal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 scale=1 1 1
- link left_central_femur: geometry collision sphere radius=0.03; visual mesh filename=package://the_walking_thread_gazebo/src/urdf/meshes/the_wal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 scale=1 1 1
- link left_central_tibia: geometry collision sphere radius=0.0065; visual mesh filename=package://the_walking_thread_gazebo/src/urdf/meshes/the_wal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 scale=1 1 1
- link left_front_coxa: geometry collision sphere radius=0.019; visual mesh filename=package://the_walking_thread_gazebo/src/urdf/meshes/the_wal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 scale=1 1 1
- link left_front_femur: geometry collision sphere radius=0.03; visual mesh filename=package://the_walking_thread_gazebo/src/urdf/meshes/the_wal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 scale=1 1 1
- link left_front_tibia: geometry collision sphere radius=0.0065; visual mesh filename=package://the_walking_thread_gazebo/src/urdf/meshes/the_wal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 scale=1 1 1
- link left_rear_coxa: geometry collision sphere radius=0.019; visual mesh filename=package://the_walking_thread_gazebo/src/urdf/meshes/the_wal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 scale=1 1 1
- link left_rear_femur: geometry collision sphere radius=0.03; visual mesh filename=package://the_walking_thread_gazebo/src/urdf/meshes/the_wal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 scale=1 1 1
- link left_rear_tibia: geometry collision sphere radius=0.0065; visual mesh filename=package://the_walking_thread_gazebo/src/urdf/meshes/the_wal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 scale=1 1 1
- link right_central_coxa: geometry collision sphere radius=0.019; visual mesh filename=package://the_walking_thread_gazebo/src/urdf/meshes/the_wal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 scale=1 1 1
- link right_central_femur: geometry collision sphere radius=0.03; visual mesh filename=package://the_walking_thread_gazebo/src/urdf/meshes/the_wal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 scale=1 1 1
- link right_central_tibia: geometry collision sphere radius=0.0065; visual mesh filename=package://the_walking_thread_gazebo/src/urdf/meshes/the_wal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 scale=1 1 1
- link right_front_coxa: geometry collision sphere radius=0.019; visual mesh filename=package://the_walking_thread_gazebo/src/urdf/meshes/the_wal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 scale=1 1 1
- link right_front_femur: geometry collision sphere radius=0.03; visual mesh filename=package://the_walking_thread_gazebo/src/urdf/meshes/the_wal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 scale=1 1 1
- link right_front_tibia: geometry collision sphere radius=0.0065; visual mesh filename=package://the_walking_thread_gazebo/src/urdf/meshes/the_wal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 scale=1 1 1
- link right_rear_coxa: geometry collision sphere radius=0.019; visual mesh filename=package://the_walking_thread_gazebo/src/urdf/meshes/the_wal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 scale=1 1 1
- link right_rear_femur: geometry collision sphere radius=0.03; visual mesh filename=package://the_walking_thread_gazebo/src/urdf/meshes/the_wal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 scale=1 1 1
- link right_rear_tibia: geometry collision sphere radius=0.0065; visual mesh filename=package://the_walking_thread_gazebo/src/urdf/meshes/the_wal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 scale=1 1 1
Joints:
- removed joint left_central_base_link_to_coxa_joint
- removed joint left_front_base_link_to_coxa_joint
- removed joint left_rear_base_link_to_coxa_joint
- removed joint right_central_base_link_to_coxa_joint
- removed joint right_front_base_link_to_coxa_joint
- removed joint right_rear_base_link_to_coxa_joint
- added joint base_link_to_body_joint: type fixed, parent base_link, child body, origin xyz=0 0 0 rpy=0 0 0
- added joint left_central_body_to_coxa_joint: type revolute, parent body, child left_central_coxa, origin xyz=0                        0.0585                        0 rpy=-1.57079632679 0 3.14159265359, axis 0 1 0, limit lower=-0.785398163397 upper=0.785398163397 effort=0.5295591 velocity=0.003141593
- added joint left_front_body_to_coxa_joint: type revolute, parent body, child left_front_coxa, origin xyz=0.1809                        0.0585                        0 rpy=-1.57079632679 0 3.14159265359, axis 0 1 0, limit lower=-0.785398163397 upper=0.785398163397 effort=0.5295591 velocity=0.003141593
- added joint left_rear_body_to_coxa_joint: type revolute, parent body, child left_rear_coxa, origin xyz=-0.1809                        0.0585                        0 rpy=-1.57079632679 0 3.14159265359, axis 0 1 0, limit lower=-0.785398163397 upper=0.785398163397 effort=0.5295591 velocity=0.003141593
- added joint right_central_body_to_coxa_joint: type revolute, parent body, child right_central_coxa, origin xyz=0                        -0.0585                        0 rpy=-1.57079632679 0 0.0, axis 0 -1 0, limit lower=-0.785398163397 upper=0.785398163397 effort=0.5295591 velocity=0.003141593
- added joint right_front_body_to_coxa_joint: type revolute, parent body, child right_front_coxa, origin xyz=0.1809                        -0.0585                        0 rpy=-1.57079632679 0 0.0, axis 0 -1 0, limit lower=-0.785398163397 upper=0.785398163397 effort=0.5295591 velocity=0.003141593
- added joint right_rear_body_to_coxa_joint: type revolute, parent body, child right_rear_coxa, origin xyz=-0.1809                        -0.0585                        0 rpy=-1.57079632679 0 0.0, axis 0 -1 0, limit lower=-0.785398163397 upper=0.785398163397 effort=0.5295591 velocity=0.003141593
